File: gripper_hat/gripper_hat/gripper_hat.kicad_pcb (KiCad board)
At the start: 4 copper layers, 65 x 30 mm, 50 parts, among them J1 GPIO, J2 SM04B-SRSS-TB(LF)(SN), J3 B2B-ZR-SM4-TF(LF)(SN), J4 5v for fan, J5 22035035, J7 pres 1, Q1 SS8550, U1 ADS1015IDGS, U2 SN74LVC1G126DBVR, U3 TPS54302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

Commit message: add pot to gripper hat pressure sense divider
Parts:
- removed R1: 110 Ohm, Resistor_SMD:R_0603_1608Metric
- added J6: extra analog breakout, Connector_Wire:SolderWire-0.25sqmm_1x02_P4.2mm_D0.65mm_OD1.7mm, F.Cu at (102.3, 91.6)
- added R2: R_Variable, easyeda2kicad:RES-ADJ-SMD_3P-L4.5-W4.5-P2.30-BL-FS, F.Cu at (118.0, 96.0)
- moved R3 11.4 mm to (128.5, 91.8), turned to -90 degrees
- moved J7 1.56 mm to (111.0, 95.7)
Connections:
- U1 pad 5: unconnected-(U1-AIN1-Pad5) -> Net-(J6-Pin_2)
Routing:
- net Net-(J6-Pin_2): track 0.00 -> 12.4 mm
- net +3V3: track 70.9 -> 77.4 mm
- net Net-(J5-Pin_3): track 26.8 -> 21.6 mm
- net Net-(J7-Pin_1): track 11.7 -> 16.6 mm
Other:
- board text added: "- ALG"
