File: gripper_hat/gripper_hat/gripper_hat.kicad_sch (KiCad schematic)
At the start: 46 parts, among them J1 GPIO, J2 SM04B-SRSS-TB(LF)(SN), J3 B2B-ZR-SM4-TF(LF)(SN), J4 5v for fan, J5 22035035, J7 pres 1, Q1 SS8550, U1 ADS1015IDGS, U2 SN74LVC1G126DBVR, U3 TPS54302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

Commit message: add pot to gripper hat pressure sense divider
Parts:
- removed R1: 110 Ohm, Resistor_SMD:R_0603_1608Metric, symbol Device:R
- added J6: extra analog breakout, Connector_Wire:SolderWire-0.25sqmm_1x02_P4.2mm_D0.65mm_OD1.7mm, symbol Connector_Generic:Conn_01x02
- added R2: R_Variable, easyeda2kicad:RES-ADJ-SMD_3P-L4.5-W4.5-P2.30-BL-FS, symbol Device:R_Variable
Connections:
- net +3V3: now also R2.2
- net GND: now also J6.1 (Pin_1)
- net at J7.1 (Pin_1), U1.4 (AIN0): now also R2.1
- net at U1.5 (AIN1): now also J6.2 (Pin_2)

Commit message: bom
Parts:
- R2: JLCPCB Part # (none) -> C124639
Changed lines of the file:
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@@
+			)
+		)
+		(property "JLCPCB Part #" "C124639"
+			(at 72.39 167.64 90)
+			(effects
+				(font
+					(size 1.27 1.27)
+				)
+				(hide yes)
 			)
 		)
