File: anchor_hat/anchor_hat/anchor_hat.kicad_sch (KiCad schematic)
At the start: 24 parts, among them J1 GPIO, J2 Motor 1, J3 Motor 2, J4 24v in barrel jack, J5 24v out slip ring, J6 5v out fan, U2 MCP2515-xST, U3 SN65HVD230, U4 TPS54302, Y1 12M

Commit message: add pinheader for alt fan plug type
Parts:
- added J7: 5v out fan right angle, Connector_PinHeader_2.54mm:PinHeader_1x02_P2.54mm_Horizontal, symbol Connector:Conn_01x02_Socket
Connections:
- net +5V: now also J7.1 (Pin_1)
- net GND: now also J7.2 (Pin_2)
