File: anchor_hat/anchor_hat/anchor_hat.kicad_pcb (KiCad board)
At the start: 4 copper layers, 65 x 30 mm, 29 parts, among them J1 GPIO, J2 Motor 1, J3 Motor 2, J4 24v in barrel jack, J5 24v out slip ring, J6 5v out fan, J7 5v out fan right angle, U2 MCP2515-xST, U3 SN65HVD230, U4 TPS54302, Y1 12M

Commit message: swap terminals on slip ring plug so ground is the lower pin
Connections:
- J5 pad 1: +24V -> GND
- J5 pad 2: GND -> +24V
Routing:
- net GND: track 53.8 -> 54.5 mm, vias 9 -> 10
Changed lines of the file:
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@@
 		(tags "connector JST ZH vertical")
 		(property "Reference" "J5"
-			(at 2.5 1.8 0)
+			(at -4.5 -3.7 0)
 			(layer "F.SilkS")
 			(effects
@@
 			(layers "F.Cu" "F.Mask" "F.Paste")
 			(roundrect_rratio 0.25)
-			(net 29 "+24V")
+			(net 1 "GND")
 			(pinfunction "Pin_1")
 			(pintype "passive")
@@
 			(layers "F.Cu" "F.Mask" "F.Paste")
 			(roundrect_rratio 0.25)
-			(net 1 "GND")
+			(net 29 "+24V")
 			(pinfunction "Pin_2")
 			(pintype "passive")
@@
 		)
 	)
-	(gr_text "24V"
-		(at 148.2 77.5 0)
+	(gr_text "GND"
+		(at 149.5 83.1 0)
 		(layer "F.SilkS")
 		(effects
@@
 	)
 	(gr_text "Slip Ring"
-		(at 152 85.1 0)
+		(at 151.9 85.2 0)
 		(layer "F.SilkS")
 		(effects
@@
 		)
 	)
-	(gr_text "Fan 5v"
-		(at 157.2 93.3 0)
+	(gr_text "24V"
+		(at 156.4 83 0)
 		(layer "F.SilkS")
 		(effects
@@
 		)
 	)
-	(gr_text "GND"
-		(at 158.1 77.565 0)
+	(gr_text "Fan 5v"
+		(at 157.2 93.3 0)
 		(layer "F.SilkS")
 		(effects
@@
 	)
 	(segment
+		(start 153.75 77.65)
+		(end 153.75 77.75)
+		(width 0.75)
+		(layer "F.Cu")
+		(net 1)
+	)
+	(segment
 		(start 121.4125 79.3375)
 		(end 121.4125 80.2125)
@@
 	)
 	(segment
-		(start 155.25 76.15)
-		(end 156.63 74.77)
-		(width 1)
+		(start 153.75 81.3)
+		(end 153.75 84.15)
+		(width 0.75)
 		(layer "F.Cu")
 		(net 1)
@@
 	)
 	(segment
-		(start 155.25 81.3)
-		(end 155.25 76.15)
-		(width 1)
-		(layer "F.Cu")
-		(net 1)
-	)
-	(segment
 		(start 121.4 79.325)
 		(end 121.4125 79.3375)
@@
 	)
 	(segment
-		(start 155.25 84.15)
-		(end 155.3 84.2)
-		(width 1)
-		(layer "F.Cu")
-		(net 1)
-	)
-	(segment
 		(start 135.33 88.4)
 		(end 135.33 86.83)
@@
 	)
 	(segment
-		(start 155.25 81.3)
-		(end 155.25 84.15)
-		(width 1)
+		(start 105.225 80.7)
+		(end 105.225 78.1)
+		(width 0.75)
 		(layer "F.Cu")
 		(net 1)
 	)
 	(segment
-		(start 105.225 80.7)
-		(end 105.225 78.1)
+		(start 153.75 77.65)
+		(end 156.63 74.77)
 		(width 0.75)
 		(layer "F.Cu")
@@
 	)
 	(segment
+		(start 153.75 81.3)
+		(end 153.75 77.65)
+		(width 0.75)
+		(layer "F.Cu")
+		(net 1)
+	)
+	(segment
 		(start 142.38 84.8)
 		(end 142.375 84.805)
@@
 	)
 	(segment
+		(start 153.75 84.15)
+		(end 153.7 84.2)
+		(width 0.75)
+		(layer "F.Cu")
+		(net 1)
+	)
+	(segment
 		(start 123.160424 85.214576)
 		(end 123.8625 84.5125)
@@
 	)
 	(via
+		(at 153.75 77.75)
+		(size 0.9)
+		(drill 0.6)
+		(layers "F.Cu" "B.Cu")
+		(net 1)
+	)
+	(via
 		(at 103.7 78.1)
 		(size 0.9)
@@
 	)
 	(via
-		(at 144.1 84.8)
+		(at 153.7 84.2)
 		(size 0.9)
 		(drill 0.6)
@@
 	)
 	(via
-		(at 103.8 79.4)
+		(at 144.1 84.8)
 		(size 0.9)
 		(drill 0.6)
@@
 	)
 	(via
-		(at 155.3 84.2)
+		(at 103.8 79.4)
 		(size 0.9)
 		(drill 0.6)
@@
 	)
 	(segment
-		(start 153.75 84.15)
-		(end 153.7 84.2)
-		(width 1)
+		(start 121.4125 84.0125)
+		(end 120.9125 84.5125)
+		(width 0.75)
 		(layer "F.Cu")
 		(net 29)
 	)
 	(segment
-		(start 153.75 81.3)
-		(end 153.75 78.65)
-		(width 1)
+		(start 120.9125 84.5125)
+		(end 120.9125 85.188044)
+		(width 0.75)
 		(layer "F.Cu")
 		(net 29)
 	)
 	(segment
-		(start 121.4125 84.0125)
-		(end 120.9125 84.5125)
+		(start 155.25 78.55)
+		(end 155.2 78.5)
 		(width 0.75)
 		(layer "F.Cu")
@@
 	)
 	(segment
-		(start 153.2 81.3)
-		(end 152.3 82.2)
-		(width 1)
+		(start 155.25 81.3)
+		(end 155.25 78.55)
+		(width 0.75)
 		(layer "F.Cu")
 		(net 29)
 	)
 	(segment
-		(start 120.9125 84.5125)
-		(end 120.9125 85.188044)
+		(start 120.9125 85.188044)
+		(end 118.080424 88.02012)
 		(width 0.75)
 		(layer "F.Cu")
@@
 	)
 	(segment
-		(start 120.9125 85.188044)
-		(end 118.080424 88.02012)
+		(start 155.25 84.15)
+		(end 155.3 84.2)
 		(width 0.75)
 		(layer "F.Cu")
@@
 	)
 	(segment
-		(start 153.75 81.3)
-		(end 153.2 81.3)
-		(width 1)
+		(start 155.8 81.3)
+		(end 156.7 82.2)
+		(width 0.75)
 		(layer "F.Cu")
 		(net 29)
 	)
 	(segment
-		(start 153.75 78.65)
-		(end 153.7 78.6)
-		(width 1)
+		(start 155.25 81.3)
+		(end 155.8 81.3)
+		(width 0.75)
 		(layer "F.Cu")
 		(net 29)
 	)
 	(segment
-		(start 153.75 81.3)
-		(end 153.75 84.15)
-		(width 1)
+		(start 155.25 81.3)
+		(end 155.25 84.15)
+		(width 0.75)
 		(layer "F.Cu")
 		(net 29)
 	)
 	(via
-		(at 152.3 82.2)
+		(at 155.2 78.5)
 		(size 0.9)
 		(drill 0.6)
@@
 	)
 	(via
-		(at 153.7 84.2)
+		(at 156.7 82.2)
 		(size 0.9)
 		(drill 0.6)
@@
 	)
 	(via
-		(at 153.7 78.6)
+		(at 155.3 84.2)
 		(size 0.9)
 		(drill 0.6)

Commit message: add elec cap to 24v rail on anchors
Parts:
- removed J6: 5v out fan, Connector_JST:JST_PH_B2B-PH-K_1x02_P2.00mm_Vertical
- added C9: 47 uf 50v, Capacitor_SMD:CP_Elec_6.3x7.7, F.Cu at (159.8, 89.1)
Routing:
- net +24V: track 14.9 -> 24.1 mm
- net GND: track 54.5 -> 60.8 mm
Other:
- board text removed: "Fan 5v"

Commit message: Layout board with mosfet, pwm fan
Parts:
- removed J7: 5v out fan right angle, Connector_PinHeader_2.54mm:PinHeader_1x02_P2.54mm_Horizontal
- added C10: 100 nf, Capacitor_SMD:C_0603_1608Metric, F.Cu at (114.8, 88.2)
- added D1: SMAJ26A, Diode_SMD:D_SMA, F.Cu at (104.4, 81.1)
- added D2: SMAJ6.0A, Diode_SMD:D_SMA, F.Cu at (115.4, 79.8)
- added J6: 5v pwm fan, Connector_JST:JST_SH_SM04B-SRSS-TB_1x04-1MP_P1.00mm_Horizontal, F.Cu at (112.6, 96.9)
- added Q1: AOD4185, Package_TO_SOT_SMD:TO-252-2, F.Cu at (136.8, 95.0)
- added Q3: 2N7002, Package_TO_SOT_SMD:SOT-23, F.Cu at (111.5, 83.6)
- added R10: 4.7kOhm, Resistor_SMD:R_1206_3216Metric, F.Cu at (138.1, 87.3)
- added R11: 560kOhm, Resistor_SMD:R_0603_1608Metric, F.Cu at (128.7, 77.2)
- added R12: 39kOhm, Resistor_SMD:R_0603_1608Metric, F.Cu at (132.0, 80.2)
- added R13: 10kOhm, Resistor_SMD:R_0603_1608Metric, F.Cu at (147.6, 77.1)
- added R14: 1kOhm, Resistor_SMD:R_0603_1608Metric, F.Cu at (114.7, 92.5)
- added R15: 100 Ohm, Resistor_SMD:R_0603_1608Metric, F.Cu at (111.5, 92.5)
- added R6: 100kOhm, Resistor_SMD:R_0603_1608Metric, F.Cu at (115.7, 86.4)
- added R7: 100kOhm, Resistor_SMD:R_0603_1608Metric, F.Cu at (114.9, 84.5)
- added R8: 10kOhm, Resistor_SMD:R_0603_1608Metric, F.Cu at (111.7, 88.2)
- added R9: 100kOhm, Resistor_SMD:R_0603_1608Metric, F.Cu at (111.7, 86.6)
- Y1: footprint easyeda2kicad:HC-49US_L11.5-W4.5-P4.88 -> Crystal:Crystal_SMD_3225-4Pin_3.2x2.5mm
- moved R4 18.5 mm to (154.1, 83.4)
- moved U3 18.1 mm to (150.3, 82.3)
- moved C3 8.09 mm to (133.6, 83.2), turned to 90 degrees
- moved R2 7.45 mm to (133.6, 80.2), turned to 90 degrees
- moved C8 7.19 mm to (144.3, 78.2), turned to 0 degrees
- moved L2 6.70 mm to (121.7, 81.2)
- moved C1 6.42 mm to (128.8, 84.9)
- moved U4 6.42 mm to (129.0, 81.5)
- moved C2 6.02 mm to (129.7, 78.8)
- moved C5 5.85 mm to (112.2, 78.7), turned to -90 degrees
- moved R5 5.28 mm to (133.3, 76.9), turned to 180 degrees
- moved R1 4.89 mm to (131.9, 83.3), turned to 90 degrees
- moved U2 4.85 mm to (138.4, 81.9)
- moved J5 3.00 mm to (157.5, 80.6)
- moved C4 2.96 mm to (109.6, 78.7), turned to -90 degrees
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Connections:
- J2 pad 1: +24V -> /+24V_MOT
- J3 pad 1: +24V -> /+24V_MOT
- U2 pad 10: unconnected-(U2-VSS-Pad10) -> GND
- U4 pad 5: unconnected-(U4-EN-Pad5) -> Net-(U4-EN)
- Y1 pad 1: Net-(U2-OSC1) -> Net-(U2-OSC2)
- Y1 pad 2: Net-(U2-OSC2) -> GND
Routing:
- net +24V: track 24.1 -> 146.3 mm, vias 3 -> 8
- net /GPIO16: track 0.00 -> 63.4 mm, vias 0 -> 1
- net /+24V_MOT: track 0.00 -> 47.0 mm
- net /GPIO12/PWM0: track 0.00 -> 45.9 mm, vias 0 -> 1
- net Net-(Q1-G): track 0.00 -> 35.0 mm, vias 0 -> 2
- net +5V: track 99.1 -> 67.8 mm, vias 2 -> 3
- net /GPIO23: track 0.00 -> 21.6 mm, vias 0 -> 1
- net GND: track 60.8 -> 79.7 mm, vias 10 -> 25
- net +3.3V: track 22.7 -> 39.6 mm, vias 1 -> 2
- net Net-(U2-OSC2): track 18.4 -> 7.00 mm
- net Net-(U2-RXCAN): track 4.93 -> 14.8 mm, vias 0 -> 2
- net Net-(U2-TXCAN): track 11.8 -> 21.3 mm, vias 0 -> 2
- net Net-(U4-EN): track 0.00 -> 6.93 mm
- net /GPIO8/SPI0.CE0: track 17.2 -> 11.9 mm
- net /GPIO10/SPI0.MOSI: track 4.79 -> 9.41 mm, vias 0 -> 1
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- added copper zone on In1.Cu, net GND
- removed copper zone on In1.Cu, net +24V
Other:
- board text added: "FAN"
- board text removed: "+5V"
- board text removed: "GND"

Commit message: V4 of anchor hat
Routing:
- net +24V: track 146.3 -> 149.3 mm
- net Net-(Q1-G): track 35.0 -> 32.5 mm
- net /+24V_MOT: track 47.0 -> 47.3 mm, vias 0 -> 8
- added copper zone on B.Cu, net /+24V_MOT
- added copper zone on F.Cu, net /+24V_MOT
Changed lines of the file:
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@@
-	)
-	(segment
-		(start 128.8925 96.3)
-		(end 120.605 88.0125)
-		(width 3)
-		(layer "F.Cu")
-		(net 17)
 	)
 	(segment
@@
 	)
 	(segment
+		(start 136.8275 96.3)
+		(end 136.8275 96.4725)
+		(width 3)
+		(layer "F.Cu")
+		(net 17)
+	)
+	(segment
+		(start 136.6 96.3)
+		(end 128.8925 96.3)
+		(width 3)
+		(layer "F.Cu")
+		(net 17)
+	)
+	(segment
+		(start 128.8925 96.3)
+		(end 120.605 88.0125)
+		(width 3)
+		(layer "F.Cu")
+		(net 17)
+	)
+	(segment
 		(start 121.4475 87.7)
 		(end 121.76 88.0125)
@@
 	)
 	(segment
+		(start 136.8275 96.4725)
+		(end 136.8 96.5)
+		(width 3)
+		(layer "F.Cu")
+		(net 17)
+	)
+	(segment
 		(start 144.405 88.7225)
 		(end 144.405 88.0125)
-		(width 3)
-		(layer "F.Cu")
-		(net 17)
-	)
-	(segment
-		(start 136.8275 96.3)
-		(end 128.8925 96.3)
 		(width 3)
 		(layer "F.Cu")
@@
 	)
 	(segment
+		(start 136.8 96.5)
+		(end 136.6 96.3)
+		(width 3)
+		(layer "F.Cu")
+		(net 17)
+	)
+	(segment
 		(start 120.455 88.1625)
 		(end 120.605 88.0125)
@@
 		(net 17)
 	)
+	(via
+		(at 137.9 96.4)
+		(size 0.9)
+		(drill 0.6)
+		(layers "F.Cu" "B.Cu")
+		(net 17)
+	)
+	(via
+		(at 128.6 96.3525)
+		(size 0.9)
+		(drill 0.6)
+		(layers "F.Cu" "B.Cu")
+		(net 17)
+	)
+	(via
+		(at 143.8 96.3525)
+		(size 0.9)
+		(drill 0.6)
+		(layers "F.Cu" "B.Cu")
+		(free yes)
+		(net 17)
+	)
+	(via
+		(at 137.9 98.1)
+		(size 0.9)
+		(drill 0.6)
+		(layers "F.Cu" "B.Cu")
+		(net 17)
+	)
+	(via
+		(at 143.8 99)
+		(size 0.9)
+		(drill 0.6)
+		(layers "F.Cu" "B.Cu")
+		(free yes)
+		(net 17)
+	)
+	(via
+		(at 128.6 99)
+		(size 0.9)
+		(drill 0.6)
+		(layers "F.Cu" "B.Cu")
+		(net 17)
+	)
+	(via
+		(at 135.6 98.1)
+		(size 0.9)
+		(drill 0.6)
+		(layers "F.Cu" "B.Cu")
+		(net 17)
+	)
+	(via
+		(at 135.6 96.4)
+		(size 0.9)
+		(drill 0.6)
+		(layers "F.Cu" "B.Cu")
+		(net 17)
+	)
 	(segment
 		(start 139.99 84.7675)
@@
 	)
 	(segment
-		(start 116.1 89.9)
-		(end 116.1 92.831371)
+		(start 137.4 92.0525)
+		(end 137.09 92.3625)
 		(width 0.3)
 		(layer "B.Cu")
@@
 	)
 	(segment
-		(start 136.1525 93.3)
-		(end 137.4 92.0525)
+		(start 137.09 92.3625)
+		(end 118.5625 92.3625)
 		(width 0.3)
 		(layer "B.Cu")
@@
 	)
 	(segment
-		(start 116.568629 93.3)
-		(end 136.1525 93.3)
-		(width 0.3)
-		(layer "B.Cu")
-		(net 28)
-	)
-	(segment
-		(start 116.1 92.831371)
-		(end 116.568629 93.3)
+		(start 118.5625 92.3625)
+		(end 116.1 89.9)
 		(width 0.3)
 		(layer "B.Cu")
@@
 	)
 	(segment
-		(start 131.8 85.2)
-		(end 134.7 88.1)
-		(width 0.75)
-		(layer "In2.Cu")
-		(net 29)
-	)
-	(segment
 		(start 117 84.3)
 		(end 117 84.8)
@@
 	)
 	(segment
+		(start 117.3 78.7)
+		(end 118.4 77.6)
+		(width 0.3)
+		(layer "In2.Cu")
+		(net 29)
+	)
+	(segment
 		(start 128.8 85.2)
-		(end 131.8 85.2)
+		(end 129.449569 85.2)
 		(width 0.75)
 		(layer "In2.Cu")
@@
 	)
 	(segment
-		(start 126.6 77.6)
-		(end 123.668629 77.6)
+		(start 117 84.3)
+		(end 117.3 84)
+		(width 0.3)
+		(layer "In2.Cu")
+		(net 29)
+	)
+	(segment
+		(start 117.3 84)
+		(end 117.3 78.7)
 		(width 0.3)
 		(layer "In2.Cu")
@@
 	)
 	(segment
+		(start 118.4 77.6)
+		(end 126.6 77.6)
+		(width 0.3)
+		(layer "In2.Cu")
+		(net 29)
+	)
+	(segment
+		(start 133.2 88.950431)
+		(end 133.2 90)
+		(width 0.75)
+		(layer "In2.Cu")
+		(net 29)
+	)
+	(segment
 		(start 111.74694 88.5875)
 		(end 117.36194 94.2025)
@@
 		(end 113.2125 88.5875)
 		(width 0.3)
+		(layer "In2.Cu")
+		(net 29)
+	)
+	(segment
+		(start 129.449569 85.2)
+		(end 133.2 88.950431)
+		(width 0.75)
 		(layer "In2.Cu")
 		(net 29)
@@
 	)
 	(segment
-		(start 123.668629 77.6)
-		(end 117 84.268629)
-		(width 0.3)
-		(layer "In2.Cu")
-		(net 29)
-	)
-	(segment
 		(start 134.7 88.1)
 		(end 134.7 92.7025)
@@
 	)
 	(zone
+		(net 17)
+		(net_name "/+24V_MOT")
+		(layer "F.Cu")
+		(hatch edge 0.5)
+		(priority 2)
+		(connect_pads yes
+			(clearance 0)
+		)
+		(min_thickness 0.25)
+		(filled_areas_thickness no)
+		(fill yes
+			(thermal_gap 0.5)
+			(thermal_bridge_width 0.5)
+		)
+		(polygon
+			(pts
+				(xy 116.7 92.8) (xy 156.6 92.8) (xy 156.6 99.9) (xy 116.7 99.8)
+			)
+		)
+	)
+	(zone
+		(net 17)
+		(net_name "/+24V_MOT")
+		(layer "B.Cu")
+		(hatch edge 0.5)
+		(priority 3)
+		(connect_pads yes
+			(clearance 0)
+		)
+		(min_thickness 0.25)
+		(filled_areas_thickness no)
+		(fill yes
+			(thermal_gap 0.5)
+			(thermal_bridge_width 0.5)
+		)
+		(polygon
+			(pts
+				(xy 116.7 92.8) (xy 116.7 99.8) (xy 156.6 99.9) (xy 156.6 92.8)
+			)
+		)
+	)
+	(zone

Commit message: replace 4 wire fan with 2 wire fan and pwm control
Parts:
- removed J6: 5v pwm fan, Connector_JST:JST_SH_SM04B-SRSS-TB_1x04-1MP_P1.00mm_Horizontal
- removed R14: 1kOhm, Resistor_SMD:R_0603_1608Metric
- removed R15: 100 Ohm, Resistor_SMD:R_0603_1608Metric
- added D3: B5819W, Diode_SMD:D_SOD-123, F.Cu at (108.9, 96.8)
- added J7: 5v pwm fan, Connector_JST:JST_PH_B2B-PH-K_1x02_P2.00mm_Vertical, F.Cu at (113.7, 95.3)
- added Q4: AO3400A, Package_TO_SOT_SMD:SOT-23, F.Cu at (113.2, 90.9)
- added R16: 100kOhm, Resistor_SMD:R_0603_1608Metric, F.Cu at (151.7, 76.9)
- R13: value 10kOhm -> 1kOhm
- moved R13 0.22 mm to (147.5, 76.9), turned to 0 degrees
Connections:
- R13 pad 1: +3.3V -> /GPIO12/PWM0
- R13 pad 2: /GPIO16 -> Net-(Q4-G)
Routing:
- net /GPIO16: track 63.4 -> 0.00 mm, vias 1 -> 0
- net Net-(Q4-G): track 0.00 -> 45.1 mm, vias 0 -> 2
- net /GPIO12/PWM0: track 45.9 -> 5.58 mm, vias 1 -> 0
- net Net-(D3-A): track 0.00 -> 13.3 mm
- net GND: track 79.7 -> 92.5 mm, vias 25 -> 21
- net Net-(J6-Pin_2): track 2.49 -> 0.00 mm
- net Net-(J6-Pin_4): track 2.49 -> 0.00 mm
- net +5V: track 67.8 -> 70.1 mm
- net +3.3V: track 39.6 -> 37.6 mm
